File: Robot-HMI/Robot-HMI.sch (KiCad schematic (older format))
At the start: 33 parts, among them J1 Conn_I2C_in, J2 Conn_I2C_out_1, SW1 SW_PUSH_1, SW2 SW_PUSH_2, SW3 SW_PUSH_3, SW4 SW_ROCKER_1, SW5 Conn_Tirette_interne, SW6 SW_reset, U1 CC56-12SRWA, U2 ProMicro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

Commit message: Robot HMI: Sync promicro and update resistences value
Parts:
- R2: value 1k -> 2.2k
- R6: value 470 -> 220
- R7: value 40k -> 39k
Changed lines of the file:
@@
 P 3950 3650
 F 0 "R2" H 4020 3696 50  0000 L CNN
-F 1 "1k" H 4020 3605 50  0000 L CNN
+F 1 "2.2k" H 4020 3605 50  0000 L CNN
 F 2 "Resistor_THT:R_Axial_DIN0207_L6.3mm_D2.5mm_P7.62mm_Horizontal" V 3880 3650 50  0001 C CNN
 F 3 "~" H 3950 3650 50  0001 C CNN
@@
 P 6200 3650
 F 0 "R6" H 6270 3696 50  0000 L CNN
-F 1 "470" H 6270 3605 50  0000 L CNN
+F 1 "220" H 6270 3605 50  0000 L CNN
 F 2 "Resistor_THT:R_Axial_DIN0207_L6.3mm_D2.5mm_P7.62mm_Horizontal" V 6130 3650 50  0001 C CNN
 F 3 "~" H 6200 3650 50  0001 C CNN
@@
 P 5100 1200
 F 0 "R7" H 5030 1154 50  0000 R CNN
-F 1 "40k" H 5030 1245 50  0000 R CNN
+F 1 "39k" H 5030 1245 50  0000 R CNN
 F 2 "Resistor_THT:R_Axial_DIN0207_L6.3mm_D2.5mm_P7.62mm_Horizontal" V 5030 1200 50  0001 C CNN
 F 3 "~" H 5100 1200 50  0001 C CNN
