File: Domotique-radiateur-controle/Domotique-radiateur-controle.kicad_pcb (KiCad board)
At the start: 2 copper layers, 50.8 x 64.8 mm, 25 parts, among them J1 Conn_01x02, J2 Conn_01x03, J3 Conn_01x04, J4 Conn_01x03, J5 Conn_01x03, U1 ESP-01v090, U2 MOC3041M, U3 MOC3041M

Commit message: Update Domotiqua radiateur controle - Add Neutre Phase Pilote indication on PCB
Other:
- board text added: "Neutre"
- board text added: "Phase"
- board text added: "Pilote"
