File: Domotique-Keyboard-et-LED-RGB/Domotique-Keyboard-et-LED-RGB.kicad_pcb (KiCad board)
At the start: 2 copper layers, 83.8 x 96.5 mm, 34 parts, among them J1 Conn_01x06, J2 Jack-DC, J3 Conn_01x04, J4 Conn_01x06, J5 Conn_01x03, J6 Conn_01x06, J7 Jack-DC, Q1 Q_NMOS_GDS, Q2 Q_NMOS_GDS, Q3 Q_NMOS_GDS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

Commit message: Domotique-Keyboard-et-LED-RGB: Version 1
Parts:
- removed H5, H6, H7, H8: MountingHole, MountingHole:MountingHole_2.2mm_M2
- removed SW7: SW_Push_SPDT, Button_Switch_THT:SW_Slide_1P2T_CK_OS102011MS2Q
- removed U4: ESP-01v090, Connector_PinHeader_2.54mm:PinHeader_2x04_P2.54mm_Vertical
- removed U5: Regulator_D24V22Fx, Pololu:Pololu_reg19a
- added A1: Arduino_Nano_v3.x, Module:Arduino_Nano, F.Cu at (115.6, 106.7)
- added J10: Conn_01x02, Connector_PinHeader_2.54mm:PinHeader_1x02_P2.54mm_Vertical, F.Cu at (90.2, 82.5)
- added J11: Conn_01x02, Connector_PinHeader_2.54mm:PinHeader_1x02_P2.54mm_Vertical, F.Cu at (81.3, 83.8)
- added J8: Conn_01x02, TerminalBlock_Phoenix:TerminalBlock_Phoenix_MKDS-1,5-2-5.08_1x02_P5.08mm_Horizontal, F.Cu at (58.4, 88.9)
- added J9: Conn_01x02, Connector_PinHeader_2.54mm:PinHeader_1x02_P2.54mm_Vertical, F.Cu at (83.8, 78.7)
- J1: footprint Connector_Molex:Molex_SL_70553-0005_1x06_P2.54mm_Horizontal -> Connector_Molex:Molex_SL_70555-0040_1x06_P2.54mm_Horizontal; moved to F.Cu
- J3: value Conn_01x04 -> Conn_PWM; footprint Connector_Molex:Molex_Micro-Fit_3.0_43650-0400_1x04_P3.00mm_Horizontal -> Connector_Molex:Molex_Micro-Fit_3.0_43650-0403_1x04_P3.00mm_Horizontal
- J4: value Conn_01x06 -> Conn_Ext_Regulator_Out_Volatage; footprint Connector_Molex:Molex_SL_70553-0005_1x06_P2.54mm_Horizontal -> Connector_PinHeader_2.54mm:PinHeader_2x02_P2.54mm_Vertical
- J5: value Conn_01x03 -> Conn_DATA; footprint Connector_Molex:Molex_Micro-Fit_3.0_43650-0300_1x03_P3.00mm_Horizontal -> Connector_Molex:Molex_Micro-Fit_3.0_43650-0303_1x04_P3.00mm_Horizontal
- J6: footprint Connector_Molex:Molex_SL_70553-0005_1x06_P2.54mm_Horizontal -> Connector_Molex:Molex_SL_70555-0040_1x06_P2.54mm_Horizontal
- J7: value Jack-DC -> Conn_Ext_Regulator; footprint TerminalBlock_Phoenix:TerminalBlock_Phoenix_MKDS-1,5-2-5.08_1x02_P5.08mm_Horizontal -> Connector_Molex:Molex_Micro-Fit_3.0_43650-0403_1x04_P3.00mm_Horizontal
- SW1: footprint Button_Switch_THT:SW_Slide_1P2T_CK_OS102011MS2Q -> Button_Switch_THT:SW_Slide_SPDT_Angled_SK12F14VG4_3mm
- U2: footprint Connector_PinHeader_2.54mm:PinHeader_2x04_P2.54mm_Vertical -> ESP8266:ESP-01
- moved J7 213.3 mm to (33.0, 101.6), turned to -90 degrees
- moved J4 202.0 mm to (35.6, 110.5), turned to 90 degrees
- moved J5 147.5 mm to (86.6, 73.5), turned to 180 degrees
- moved U2 71.2 mm to (104.1, 91.4), turned to 0 degrees
- moved J1 64.5 mm to (94.0, 103.4), turned to 0 degrees
- moved H4 59.1 mm to (120.7, 71.1)
- moved H3 57.2 mm to (120.7, 109.2)
- moved SW1 39.9 mm to (65.8, 111.0), turned to 0 degrees
- moved J3 38.6 mm to (66.7, 73.7)
- moved U1 36.2 mm to (51.4, 105.4), turned to -90 degrees
- moved Q3 33.1 mm to (84.5, 94.0)
- moved H1 20.4 mm to (29.2, 83.8)
- moved J2 18.3 mm to (45.7, 88.9)
- moved Q2 17.0 mm to (68.6, 83.8)
- moved Q1 15.5 mm to (68.6, 97.8)
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Connections:
- net /RGB1_BLUE renamed /RGB_BLUE
- net /RGB1_GREEN renamed /RGB_GREEN
- net /RGB1_PROG_3.3V renamed /RGB_PROG_3.3V
- net /RGB1_RED renamed /RGB_RED
- net /RGB1_RESET renamed /RGB_RESET
- net /RGB1_TX renamed /RGB_TX
- net Net-(SW1-Pad2) renamed /RGB_3.3V
- J1 pad 1: /RGB1_GND -> /RGB_GND
- J2 pad 1: /RGB1_5V -> /RGB_IN_GND
- J2 pad 2: /RGB1_GND -> /RGB_VIN
- J3 pad 1: /RGB1_5V -> /RGB_VIN
- J4 pad 1: /RGB2_GND -> Net-(J4-Pin_1)
- J4 pad 2: /RGB2_PROG_3.3V -> Net-(J4-Pin_1)
- J4 pad 3: /RGB2_TX -> /RGB_REG_3.3V
- J4 pad 4: /RGB2_DATA -> /RGB_5V
- J5 pad 1: /RGB2_GND -> /RGB_GND
- J5 pad 2: /RGB2_DATA -> /RGB_DATA
- J5 pad 3: /RGB2_5V -> Net-(J5-Pin_3)
- J7 pad 1: /RGB2_5V -> /RGB_GND
- J7 pad 2: /RGB2_GND -> Net-(J4-Pin_1)
- Q1 pad 3: /RGB1_GND -> /RGB_IN_GND
- Q2 pad 3: /RGB1_GND -> /RGB_IN_GND
- Q3 pad 3: /RGB1_GND -> /RGB_IN_GND
- SW1 pad 1: /RGB1_3.3V -> /RGB_REG_3.3V
- U1 pad 1: Net-(U1-Pad1) -> unconnected-(U1-PG-Pad1)
- U1 pad 2: Net-(U1-Pad2) -> unconnected-(U1-EN-Pad2)
- U1 pad 3: /RGB1_5V -> /RGB_VIN
- U1 pad 4: /RGB1_GND -> /RGB_IN_GND
- U1 pad 5: /RGB1_3.3V -> /RGB_REG_3.3V
- U1 pad 6: /RGB1_GND -> /RGB_GND
- U2 pad 2: /RGB1_GND -> /RGB_GND
- U2 pad 3: Net-(U2-Pad3) -> unconnected-(U2-CH_PD-Pad3)
- U3 pad 1: Net-(U3-Pad1) -> unconnected-(U3-1/TX-Pad1)
- U3 pad 11: Net-(U3-Pad11) -> unconnected-(U3-8/B4-Pad11)
- U3 pad 12: Net-(U3-Pad12) -> unconnected-(U3-9/B5-Pad12)
- U3 pad 13: Net-(U3-Pad13) -> unconnected-(U3-10/B6-Pad13)
- U3 pad 17: Net-(U3-Pad17) -> unconnected-(U3-A0/F7-Pad17)
- U3 pad 18: Net-(U3-Pad18) -> unconnected-(U3-A1/F6-Pad18)
- U3 pad 19: Net-(U3-Pad19) -> unconnected-(U3-A2/F5-Pad19)
- U3 pad 2: Net-(U3-Pad2) -> unconnected-(U3-0/RX-Pad2)
- U3 pad 20: Net-(U3-Pad20) -> unconnected-(U3-A3/F4-Pad20)
- U3 pad 21: Net-(U3-Pad21) -> unconnected-(U3-VCC-Pad21)
- U3 pad 3: Net-(U3-Pad3) -> unconnected-(U3-GND-Pad3)
- U3 pad 5: Net-(U3-Pad5) -> unconnected-(U3-2/SDA-Pad5)
Routing:
- net /RGB_GND: track 0.00 -> 153.3 mm
- net /RGB_IN_GND: track 0.00 -> 99.4 mm
- net /RGB_3.3V: track 0.00 -> 95.6 mm
- net /RGB_GREEN: track 0.00 -> 87.6 mm, vias 0 -> 1
- net /RGB_RED: track 0.00 -> 82.4 mm
- net /RGB_VIN: track 0.00 -> 74.9 mm
- net /RGB_5V: track 0.00 -> 65.9 mm, vias 0 -> 1
- net /RGB_RESET: track 0.00 -> 59.0 mm, vias 0 -> 2
- net /RGB_TX: track 0.00 -> 58.1 mm, vias 0 -> 1
- net /RGB_BLUE: track 0.00 -> 52.7 mm
- net /RGB_REG_3.3V: track 0.00 -> 49.7 mm
- net /RGB_DATA: track 0.00 -> 43.8 mm
- net Net-(J3-Pin_2): track 0.00 -> 28.8 mm
- net Net-(J3-Pin_4): track 0.00 -> 26.5 mm
- net /RGB_PROG_3.3V: track 0.00 -> 24.3 mm
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Other:
- board size 83.8 x 96.5 mm -> 99.1 x 88.9 mm
- net class Default removed
- board text added: "10/2024 V1"
- board text added: "3.3V"
- board text added: "5V"
- board text added: "GND"
- board text added: "Red/Data"
- board text added: "VIN"
