File: ebike-can-monitor/ebike-can-monitor.kicad_pcb (KiCad board)
At the start: 2 copper layers, 76.2 x 27.9 mm, 30 parts, among them J1 Conn_01x05, J2 Conn_01x05, J3 Conn_01x02, SW1 SW_SPDT, U1 XIAO-ESP32-C6-SMD, U2 SN65HVD230, U4 LV2862XLVDDCR

Commit message: ebike-monitor: Fix diode
Parts:
- moved D1 0.51 mm to (109.3, 34.2), turned to -90 degrees
Connections:
- C1 pad 2: Net-(D1-A) -> Net-(D1-K)
- D1 pad 1: GND -> Net-(D1-K)
- D1 pad 2: Net-(D1-A) -> GND
- L1 pad 1: Net-(D1-A) -> Net-(D1-K)
- U4 pad 6: Net-(D1-A) -> Net-(D1-K)
Routing:
- net Net-(D1-K): track 0.00 -> 24.0 mm
- net Net-(D1-A): track 24.0 -> 0.00 mm
- net GND: track 105.8 -> 105.2 mm
Other:
- board text added: "BAT"
- board text added: "USB"
